Commit message: nav_to_pose (avoid obstacle): doing

File: src/lower_layer_mvibot/urdf/fcr.urdf (robot description, URDF)
Before this commit: robot mvibot, 8 links, 7 joints
Joints:
- joint base_lidar_1: origin xyz=0.392 0.241 0.222 rpy=0 0 ${-pi/2} -> xyz=0.415 0.241 0.222 rpy=0 0 ${-pi/2}
- joint base_lidar_2: origin xyz=-0.546 -0.24 0.222 rpy=0 0 ${pi/2} -> xyz=-0.555 -0.24 0.222 rpy=0 0 ${pi/2}
- joint camera1: origin xyz=0.438 -0.126 0.411 rpy=${-pi/2} 0 ${pi/9} -> xyz=0.46 0.126 0.411 rpy=${-pi/2} 0 ${-pi/9}
- joint camera2: origin xyz=0.438 0.126 0.411 rpy=${-pi/2} 0 ${-pi/9} -> xyz=0.46 -0.126 0.411 rpy=${-pi/2} 0 ${pi/9}

Commit message: reset  mission

File: src/lower_layer_mvibot/urdf/fcr.urdf (robot description, URDF)
Before this commit: robot mvibot, 8 links, 7 joints
Joints:
- joint camera1: origin xyz=0.46 0.126 0.411 rpy=${-pi/2} 0 ${-pi/9} -> xyz=0.46 0.126 0.38 rpy=${-pi/2} 0 ${-pi/9}
- joint camera2: origin xyz=0.46 -0.126 0.411 rpy=${-pi/2} 0 ${pi/9} -> xyz=0.46 -0.126 0.38 rpy=${-pi/2} 0 ${pi/9}

Commit message: fix display led, coverage area with long h

File: src/lower_layer_mvibot/urdf/fcr.urdf (robot description, URDF)
Before this commit: robot mvibot, 8 links, 7 joints
Joints:
- joint base_lidar_1: origin xyz=0.415 0.241 0.222 rpy=0 0 ${-pi/2} -> xyz=0.415 0.241 0.22 rpy=0 0 ${-pi/2}
- joint base_lidar_2: origin xyz=-0.555 -0.24 0.222 rpy=0 0 ${pi/2} -> xyz=-0.555 -0.24 0.22 rpy=0 0 ${pi/2}

Commit message: update config moshi

File: src/lower_layer_mvibot/urdf/fcr.urdf (robot description, URDF)
Before this commit: robot mvibot, 8 links, 7 joints
Joints:
- joint base_lidar_2: origin xyz=-0.555 -0.24 0.22 rpy=0 0 ${pi/2} -> xyz=-0.555 -0.24 0.2 rpy=0 0 ${pi/2}

Commit message: feat: scan wifi and apriltag marker

File: src/lower_layer_mvibot/urdf/fcr.urdf (robot description, URDF)
Before this commit: robot mvibot, 8 links, 7 joints
Links:
- added link $(arg mvibot_seri)/camera
Joints:
- added joint camera: type fixed, parent $(arg mvibot_seri)/base_link, child $(arg mvibot_seri)/camera, origin xyz=-0.65 0.0 0.54 rpy=${-pi/2} 0 ${pi/2}
