Commit message: fix: control water valve, feat: preview path when zoning

File: install/realsense2_description/share/realsense2_description/urdf/_d405.urdf.xacro (robot description, xacro)
@@ -1 +1 @@
-/home/mvibot/floorCleaningRobot_ws/src/floorCleaningRobot_ws/src/realsense-ros/realsense2_description/urdf/_d405.urdf.xacro
+/home/mvibot/floorCleaningRobot_ws/src/realsense-ros/realsense2_description/urdf/_d405.urdf.xacro

File: install/realsense2_description/share/realsense2_description/urdf/_d415.urdf.xacro (robot description, xacro)
@@ -1 +1 @@
-/home/mvibot/floorCleaningRobot_ws/src/floorCleaningRobot_ws/src/realsense-ros/realsense2_description/urdf/_d415.urdf.xacro
+/home/mvibot/floorCleaningRobot_ws/src/realsense-ros/realsense2_description/urdf/_d415.urdf.xacro

File: install/realsense2_description/share/realsense2_description/urdf/_d435.urdf.xacro (robot description, xacro)
@@ -1 +1 @@
-/home/mvibot/floorCleaningRobot_ws/src/floorCleaningRobot_ws/src/realsense-ros/realsense2_description/urdf/_d435.urdf.xacro
+/home/mvibot/floorCleaningRobot_ws/src/realsense-ros/realsense2_description/urdf/_d435.urdf.xacro

File: install/realsense2_description/share/realsense2_description/urdf/_d435i.urdf.xacro (robot description, xacro)
@@ -1 +1 @@
-/home/mvibot/floorCleaningRobot_ws/src/floorCleaningRobot_ws/src/realsense-ros/realsense2_description/urdf/_d435i.urdf.xacro
+/home/mvibot/floorCleaningRobot_ws/src/realsense-ros/realsense2_description/urdf/_d435i.urdf.xacro

File: install/realsense2_description/share/realsense2_description/urdf/_d435i_imu_modules.urdf.xacro (robot description, xacro)
@@ -1 +1 @@
-/home/mvibot/floorCleaningRobot_ws/src/floorCleaningRobot_ws/src/realsense-ros/realsense2_description/urdf/_d435i_imu_modules.urdf.xacro
+/home/mvibot/floorCleaningRobot_ws/src/realsense-ros/realsense2_description/urdf/_d435i_imu_modules.urdf.xacro

File: install/realsense2_description/share/realsense2_description/urdf/_d455.urdf.xacro (robot description, xacro)
@@ -1 +1 @@
-/home/mvibot/floorCleaningRobot_ws/src/floorCleaningRobot_ws/src/realsense-ros/realsense2_description/urdf/_d455.urdf.xacro
+/home/mvibot/floorCleaningRobot_ws/src/realsense-ros/realsense2_description/urdf/_d455.urdf.xacro

File: install/realsense2_description/share/realsense2_description/urdf/_materials.urdf.xacro (robot description, xacro)
@@ -1 +1 @@
-/home/mvibot/floorCleaningRobot_ws/src/floorCleaningRobot_ws/src/realsense-ros/realsense2_description/urdf/_materials.urdf.xacro
+/home/mvibot/floorCleaningRobot_ws/src/realsense-ros/realsense2_description/urdf/_materials.urdf.xacro

File: install/realsense2_description/share/realsense2_description/urdf/_r410.urdf.xacro (robot description, xacro)
@@ -1 +1 @@
-/home/mvibot/floorCleaningRobot_ws/src/floorCleaningRobot_ws/src/realsense-ros/realsense2_description/urdf/_r410.urdf.xacro
+/home/mvibot/floorCleaningRobot_ws/src/realsense-ros/realsense2_description/urdf/_r410.urdf.xacro

File: install/realsense2_description/share/realsense2_description/urdf/_r430.urdf.xacro (robot description, xacro)
@@ -1 +1 @@
-/home/mvibot/floorCleaningRobot_ws/src/floorCleaningRobot_ws/src/realsense-ros/realsense2_description/urdf/_r430.urdf.xacro
+/home/mvibot/floorCleaningRobot_ws/src/realsense-ros/realsense2_description/urdf/_r430.urdf.xacro

File: install/realsense2_description/share/realsense2_description/urdf/_usb_plug.urdf.xacro (robot description, xacro)
@@ -1 +1 @@
-/home/mvibot/floorCleaningRobot_ws/src/floorCleaningRobot_ws/src/realsense-ros/realsense2_description/urdf/_usb_plug.urdf.xacro
+/home/mvibot/floorCleaningRobot_ws/src/realsense-ros/realsense2_description/urdf/_usb_plug.urdf.xacro

File: install/realsense2_description/share/realsense2_description/urdf/test_d405_camera.urdf.xacro (robot description, xacro)
@@ -1 +1 @@
-/home/mvibot/floorCleaningRobot_ws/src/floorCleaningRobot_ws/src/realsense-ros/realsense2_description/urdf/test_d405_camera.urdf.xacro
+/home/mvibot/floorCleaningRobot_ws/src/realsense-ros/realsense2_description/urdf/test_d405_camera.urdf.xacro

File: install/realsense2_description/share/realsense2_description/urdf/test_d415_camera.urdf.xacro (robot description, xacro)
@@ -1 +1 @@
-/home/mvibot/floorCleaningRobot_ws/src/floorCleaningRobot_ws/src/realsense-ros/realsense2_description/urdf/test_d415_camera.urdf.xacro
+/home/mvibot/floorCleaningRobot_ws/src/realsense-ros/realsense2_description/urdf/test_d415_camera.urdf.xacro

File: install/realsense2_description/share/realsense2_description/urdf/test_d435_camera.urdf.xacro (robot description, xacro)
@@ -1 +1 @@
-/home/mvibot/floorCleaningRobot_ws/src/floorCleaningRobot_ws/src/realsense-ros/realsense2_description/urdf/test_d435_camera.urdf.xacro
+/home/mvibot/floorCleaningRobot_ws/src/realsense-ros/realsense2_description/urdf/test_d435_camera.urdf.xacro

File: install/realsense2_description/share/realsense2_description/urdf/test_d435_multiple_cameras.urdf.xacro (robot description, xacro)
@@ -1 +1 @@
-/home/mvibot/floorCleaningRobot_ws/src/floorCleaningRobot_ws/src/realsense-ros/realsense2_description/urdf/test_d435_multiple_cameras.urdf.xacro
+/home/mvibot/floorCleaningRobot_ws/src/realsense-ros/realsense2_description/urdf/test_d435_multiple_cameras.urdf.xacro

File: install/realsense2_description/share/realsense2_description/urdf/test_d435i_camera.urdf.xacro (robot description, xacro)
@@ -1 +1 @@
-/home/mvibot/floorCleaningRobot_ws/src/floorCleaningRobot_ws/src/realsense-ros/realsense2_description/urdf/test_d435i_camera.urdf.xacro
+/home/mvibot/floorCleaningRobot_ws/src/realsense-ros/realsense2_description/urdf/test_d435i_camera.urdf.xacro

File: install/realsense2_description/share/realsense2_description/urdf/test_d455_camera.urdf.xacro (robot description, xacro)
@@ -1 +1 @@
-/home/mvibot/floorCleaningRobot_ws/src/floorCleaningRobot_ws/src/realsense-ros/realsense2_description/urdf/test_d455_camera.urdf.xacro
+/home/mvibot/floorCleaningRobot_ws/src/realsense-ros/realsense2_description/urdf/test_d455_camera.urdf.xacro

File: install/realsense2_description/share/realsense2_description/urdf/test_r410_camera.urdf.xacro (robot description, xacro)
@@ -1 +1 @@
-/home/mvibot/floorCleaningRobot_ws/src/floorCleaningRobot_ws/src/realsense-ros/realsense2_description/urdf/test_r410_camera.urdf.xacro
+/home/mvibot/floorCleaningRobot_ws/src/realsense-ros/realsense2_description/urdf/test_r410_camera.urdf.xacro

File: install/realsense2_description/share/realsense2_description/urdf/test_r430_camera.urdf.xacro (robot description, xacro)
@@ -1 +1 @@
-/home/mvibot/floorCleaningRobot_ws/src/floorCleaningRobot_ws/src/realsense-ros/realsense2_description/urdf/test_r430_camera.urdf.xacro
+/home/mvibot/floorCleaningRobot_ws/src/realsense-ros/realsense2_description/urdf/test_r430_camera.urdf.xacro

File: src/lower_layer_mvibot/urdf/fcr.urdf (robot description, URDF)
Before this commit: robot mvibot, 9 links, 8 joints
Joints:
- joint camera1: origin xyz=0.46 0.126 0.38 rpy=${-pi/2} 0 ${-pi/9} -> xyz=0.48 0.126 0.36 rpy=${-pi/2} 0 ${-pi/9}
- joint camera2: origin xyz=0.46 -0.126 0.38 rpy=${-pi/2} 0 ${pi/9} -> xyz=0.48 -0.126 0.36 rpy=${-pi/2} 0 ${pi/9}
